File: pov-globe2.brd (EAGLE design)
At the start: 96.4 x 101.6 mm, 82 parts, among them IC1 74595, IC2 74595, IC3 74595, IC4 MEGA8-AI, IC5 REG1117, IC6 74595, IC7 74595

Commit message: more updates
Parts:
- C10: device rcl:E2-5 -> rcl:C0805
- C14: device rcl:C0805 -> rcl:E2-5
- IC1: value 74595 -> MEGA8-AI; device SparkFun:TSSOP16 -> atmel:TQFP32-08
- IC2: value 74595 -> REG1117; device SparkFun:TSSOP16 -> burr-brown:SOT223
- IC4: value MEGA8-AI -> 74595; device atmel:TQFP32-08 -> SparkFun:TSSOP16
- IC5: value REG1117 -> 74595; device burr-brown:SOT223 -> SparkFun:TSSOP16
- moved C10 46.7 mm to (47.8, 34.5), turned to 270 degrees
- moved C14 46.3 mm to (61.8, 80.4)
- moved IC1 40.4 mm to (61.0, 43.7), turned to 0 degrees
- moved C15 33.5 mm to (67.3, 43.2), turned to 270 degrees
- moved IC4 30.7 mm to (37.3, 63.2), turned to 270 degrees
- moved IC5 30.6 mm to (37.3, 50.0)
- moved C9 27.5 mm to (47.8, 40.6), turned to 90 degrees
- moved IC3 26.4 mm to (37.3, 76.5)
- moved IC2 24.4 mm to (61.0, 69.5)
- moved C7 22.5 mm to (61.0, 64.8), turned to 180 degrees
- moved C5 12.2 mm to (37.5, 27.9), turned to 0 degrees
- moved C4 10.4 mm to (37.3, 41.1), turned to 0 degrees
- moved C13 5.84 mm to (56.0, 80.5)
- renumbered JP1 to SERIALPROG, LED25 to DIAG, Q1 to X1, R26 to R1, S2 to A, S3 to B, S4 to C, U$1 to ICSP
Connections:
- net +12V: now also C13.+, C7.2, IC2.3; no longer C10.+, C9.2, IC5.3
- net +5V: now also C14.+, C4.2, C5.2, IC1.18, IC1.20, IC1.4, IC1.6, IC2.2, IC4.10, IC4.16, IC5.10, IC5.16; no longer C13.+, C14.2, C7.2, IC1.10, IC1.16, IC2.10, IC2.16, IC4.18, IC4.20, IC4.4, IC4.6, IC5.2
- net DIAG: now also IC1.17; no longer IC4.17
- net EN_LEDS: now also IC1.10, IC4.13, IC5.13; no longer IC1.13, IC2.13, IC4.10
- net GND: now also C10.1, C14.-, IC1.21, IC1.3, IC1.5, IC2.1, IC4.8, IC5.8; no longer C10.-, C14.1, IC1.8, IC2.8, IC4.21, IC4.3, IC4.5, IC5.1
- net N$13: now also IC3.4; no longer IC1.4
- net N$14: now also IC3.5; no longer IC1.5
- net N$15: now also IC3.6; no longer IC1.6
- net N$16: now also IC3.7; no longer IC1.7
- net N$17: now also IC1.31; no longer IC4.31
- net N$18: now also IC1.30; no longer IC4.30
- net N$19: now also IC1.16; no longer IC4.16
- net N$21: now also IC1.15; no longer IC4.15
- net N$27: now also IC4.15; no longer IC2.15
- net N$28: now also IC4.1; no longer IC2.1
- net N$29: now also IC4.2; no longer IC2.2
- net N$30: now also IC4.3; no longer IC2.3
- net N$35: now also IC4.4; no longer IC2.4
- net N$36: now also IC4.5; no longer IC2.5
- net N$37: now also IC4.6; no longer IC2.6
- net N$38: now also IC1.29; no longer IC4.29
- net N$40: now also IC4.7; no longer IC2.7
- net N$45: now also IC5.15; no longer IC3.15
- net N$46: now also IC5.1; no longer IC3.1
- net N$47: now also IC5.2; no longer IC3.2
- net N$48: now also IC5.3; no longer IC3.3
- net N$5: now also IC3.15; no longer IC1.15
- net N$53: now also IC5.4; no longer IC3.4
- net N$54: now also IC5.5; no longer IC3.5
- net N$55: now also IC5.6; no longer IC3.6
- net N$56: now also IC5.7; no longer IC3.7
- net N$59: now also C9.2, IC1.7; no longer C4.2, IC4.7
- net N$6: now also IC3.1; no longer IC1.1
- net N$60: now also C10.2, IC1.8; no longer C5.2, IC4.8
- net N$7: now also IC3.2; no longer IC1.2
- net N$8: now also IC3.3; no longer IC1.3
- net RCK: now also IC1.9, IC4.12, IC5.12; no longer IC1.12, IC2.12, IC4.9
- net SCK: now also IC1.2, IC4.11, IC5.11; no longer IC1.11, IC2.11, IC4.2
- net SENSOR: now also IC1.32; no longer IC4.32
- net SER1: now also IC1.23, IC3.14; no longer IC1.14, IC4.23
- net SER2: now also IC1.24, IC4.14; no longer IC2.14, IC4.24
- net SER3: now also IC1.25, IC5.14; no longer IC3.14, IC4.25
- net SER4: now also IC1.26; no longer IC4.26
- net SER5: now also IC1.27; no longer IC4.27
- net SWITCH1: now also IC1.12; no longer IC4.12
- net SWITCH2: now also IC1.13; no longer IC4.13
- net SWITCH3: now also IC1.14; no longer IC4.14
Routing:
- net +5V: track 272.5 -> 275.6 mm
- net N$85: track 6.22 -> 7.22 mm
- net N$86: track 5.30 -> 6.05 mm
- net N$87: track 4.46 -> 4.98 mm
Other:
- board text added: "1"

Commit message: pcb rev1
Parts:
- IC2: value REG1117 -> 7805DT; device burr-brown:SOT223 -> linear:TO252
- moved S1 89.5 mm to (70.1, 10.9), turned to 115 degrees
- moved C8 86.6 mm to (71.3, 12.8), turned to 0 degrees
- moved C7 10.9 mm to (57.1, 74.9)
- moved C6 9.67 mm to (57.1, 65.3)
- moved IC2 0.71 mm to (61.0, 70.2)
Connections:
- net +12V: now also IC2.1; no longer IC2.3
- net GND: now also IC2.3; no longer IC2.1
Routing:
- net +12V: track 47.3 -> 36.0 mm
- net GND: track 184.8 -> 174.4 mm
- net +5V: track 275.6 -> 282.1 mm, vias 14 -> 15
- net SENSOR: track 70.8 -> 68.4 mm
Other:
- board size 96.4 x 101.6 mm -> 96.4 x 105.5 mm
- board text added: "GLOBE"
- board text added: "POV"
- board text added: "hotchk155"
- board text added: "rev 1"
