File: pov-globe2.brd (EAGLE design)
At the start: 96.4 x 100.1 mm, 82 parts, among them IC1 MEGA8-AI, IC2 7805DT, IC3 74595, IC4 74595, IC5 74595, IC6 74595, IC7 74595

Commit message: slot routing2
Routing:
- net +12V: track 36.0 -> 8.56 mm
- net GND: track 174.4 -> 150.1 mm
- net +5V: track 282.5 -> 268.7 mm
Other:
- outline, holes or cut-outs redrawn
- board text added: "rev 2"
- board text removed: "rev 1"
