File: pov-globe2.sch (EAGLE design)
At the start: 82 parts, among them IC1 74595, IC2 74595, IC3 74595, IC4 MEGA8-AI, IC5 REG1117, IC6 74595, IC7 74595

Commit message: more updates
Parts:
- C10: device rcl:CPOL-EUE2-5 -> rcl:C-EUC0805
- C14: device rcl:C-EUC0805 -> rcl:CPOL-EUE2-5
- IC1: value 74595 -> MEGA8-AI; device SparkFun:74595 -> atmel:MEGA8-AI
- IC2: value 74595 -> REG1117; device SparkFun:74595 -> burr-brown:REG1117
- IC4: value MEGA8-AI -> 74595; device atmel:MEGA8-AI -> SparkFun:74595
- IC5: value REG1117 -> 74595; device burr-brown:REG1117 -> SparkFun:74595
- renumbered JP1 to SERIALPROG, LED25 to DIAG, Q1 to X1, R26 to R1, S2 to A, S3 to B, S4 to C, U$1 to ICSP
Connections:
- net +12V: now also C13.+, C7.2, IC2.VIN; no longer C10.+, C9.2, IC5.VIN
- net +5V: now also C14.+, C4.2, C5.2, IC1.AREF, IC1.AVCC, IC1.VCC@1, IC1.VCC@2, IC2.VOUT, IC4.SCL, IC4.VCC, IC5.SCL, IC5.VCC; no longer C13.+, C14.2, C7.2, IC1.SCL, IC1.VCC, IC2.SCL, IC2.VCC, IC4.AREF, IC4.AVCC, IC4.VCC@1, IC4.VCC@2, IC5.VOUT
- net DIAG: now also IC1.PB5(SCK); no longer IC4.PB5(SCK)
- net EN_LEDS: now also IC1.PD6(AIN0), IC4.G, IC5.G; no longer IC1.G, IC2.G, IC4.PD6(AIN0)
- net GND: now also C10.1, C14.-, IC1.GND@1, IC1.GND@2; no longer C10.-, C14.1, IC4.GND@1, IC4.GND@2
- net N$13: now also IC3.QE; no longer IC1.QE
- net N$14: now also IC3.QF; no longer IC1.QF
- net N$15: now also IC3.QG; no longer IC1.QG
- net N$16: now also IC3.QH; no longer IC1.QH
- net N$17: now also IC1.PD1(TXD); no longer IC4.PD1(TXD)
- net N$18: now also IC1.PD0(RXD); no longer IC4.PD0(RXD)
- net N$19: now also IC1.PB4(MISO); no longer IC4.PB4(MISO)
- net N$21: now also IC1.PB3(MOSI/OC2); no longer IC4.PB3(MOSI/OC2)
- net N$27: now also IC4.QA; no longer IC2.QA
- net N$28: now also IC4.QB; no longer IC2.QB
- net N$29: now also IC4.QC; no longer IC2.QC
- net N$30: now also IC4.QD; no longer IC2.QD
- net N$35: now also IC4.QE; no longer IC2.QE
- net N$36: now also IC4.QF; no longer IC2.QF
- net N$37: now also IC4.QG; no longer IC2.QG
- net N$38: now also IC1.PC6(/RESET); no longer IC4.PC6(/RESET)
- net N$40: now also IC4.QH; no longer IC2.QH
- net N$45: now also IC5.QA; no longer IC3.QA
- net N$46: now also IC5.QB; no longer IC3.QB
- net N$47: now also IC5.QC; no longer IC3.QC
- net N$48: now also IC5.QD; no longer IC3.QD
- net N$5: now also IC3.QA; no longer IC1.QA
- net N$53: now also IC5.QE; no longer IC3.QE
- net N$54: now also IC5.QF; no longer IC3.QF
- net N$55: now also IC5.QG; no longer IC3.QG
- net N$56: now also IC5.QH; no longer IC3.QH
- net N$59: now also C9.2, IC1.PB6(XTAL1/TOSC1); no longer C4.2, IC4.PB6(XTAL1/TOSC1)
- net N$6: now also IC3.QB; no longer IC1.QB
- net N$60: now also C10.2, IC1.PB7(XTAL2/TOSC2); no longer C5.2, IC4.PB7(XTAL2/TOSC2)
- net N$7: now also IC3.QC; no longer IC1.QC
- net N$8: now also IC3.QD; no longer IC1.QD
- net RCK: now also IC1.PD5(T1), IC4.RCK, IC5.RCK; no longer IC1.RCK, IC2.RCK, IC4.PD5(T1)
- net SCK: now also IC1.PD4(XCK/T0), IC4.SCK, IC5.SCK; no longer IC1.SCK, IC2.SCK, IC4.PD4(XCK/T0)
- net SENSOR: now also IC1.PD2(INT0); no longer IC4.PD2(INT0)
- net SER1: now also IC1.PC0(ADC0), IC3.SER; no longer IC1.SER, IC4.PC0(ADC0)
- net SER2: now also IC1.PC1(ADC1), IC4.SER; no longer IC2.SER, IC4.PC1(ADC1)
- net SER3: now also IC1.PC2(ADC2), IC5.SER; no longer IC3.SER, IC4.PC2(ADC2)
- net SER4: now also IC1.PC3(ADC3); no longer IC4.PC3(ADC3)
- net SER5: now also IC1.PC4(ADC4/SDA); no longer IC4.PC4(ADC4/SDA)
- net SWITCH1: now also IC1.PB0(ICP); no longer IC4.PB0(ICP)
- net SWITCH2: now also IC1.PB1(OC1A); no longer IC4.PB1(OC1A)
- net SWITCH3: now also IC1.PB2(SS/OC1B); no longer IC4.PB2(SS/OC1B)
Other:
- moved on the sheet: C13, C15, C4, C5, C7, C9, IC3

Commit message: pcb rev1
Parts:
- IC2: value REG1117 -> 7805DT; device burr-brown:REG1117 -> linear:7805DT
Connections:
- net +12V: now also IC2.VI; no longer IC2.VIN
- net +5V: now also IC2.VO; no longer IC2.VOUT
Changed lines of the file:
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@@
 <part name="SUPPLY6" library="supply2" deviceset="GND" device=""/>
 <part name="C15" library="rcl" deviceset="C-EU" device="C0805"/>
-<part name="IC2" library="burr-brown" deviceset="REG1117" device=""/>
 <part name="SUPPLY7" library="supply2" deviceset="GND" device=""/>
 <part name="SUPPLY8" library="supply2" deviceset="+5V" device=""/>
@@
 <part name="SUPPLY26" library="supply2" deviceset="GND" device=""/>
 <part name="RESET" library="switch-omron" deviceset="10-XX" device=""/>
+<part name="IC2" library="linear" deviceset="78*" device="DT" technology="05"/>
 </parts>
 <sheets>
@@
 <instance part="SUPPLY6" gate="GND" x="-175.26" y="33.02"/>
 <instance part="C15" gate="G$1" x="-175.26" y="43.18" rot="R180"/>
-<instance part="IC2" gate="G$1" x="-182.88" y="7.62"/>
 <instance part="SUPPLY7" gate="GND" x="-182.88" y="-12.7"/>
 <instance part="SUPPLY8" gate="+5V" x="-160.02" y="17.78"/>
@@
 <instance part="SUPPLY26" gate="GND" x="109.22" y="-76.2"/>
 <instance part="RESET" gate="1" x="-111.76" y="76.2" rot="R270"/>
+<instance part="IC2" gate="A1" x="-182.88" y="7.62"/>
 </instances>
 <busses>
@@
 </segment>
 <segment>
-<pinref part="IC2" gate="G$1" pin="VOUT"/>
 <pinref part="SUPPLY8" gate="+5V" pin="+5V"/>
 <wire x1="-170.18" y1="7.62" x2="-167.64" y2="7.62" width="0.1524" layer="91"/>
@@
 <wire x1="-160.02" y1="5.08" x2="-160.02" y2="7.62" width="0.1524" layer="91"/>
 <junction x="-160.02" y="7.62"/>
+<pinref part="IC2" gate="A1" pin="VO"/>
+<wire x1="-172.72" y1="7.62" x2="-170.18" y2="7.62" width="0.1524" layer="91"/>
 </segment>
 <segment>
@@
 </segment>
 <segment>
-<pinref part="IC2" gate="G$1" pin="GND"/>
 <pinref part="SUPPLY7" gate="GND" pin="GND"/>
 <wire x1="-182.88" y1="-5.08" x2="-182.88" y2="-7.62" width="0.1524" layer="91"/>
@@
 <wire x1="-198.12" y1="-2.54" x2="-198.12" y2="-7.62" width="0.1524" layer="91"/>
 <junction x="-198.12" y="-7.62"/>
+<pinref part="IC2" gate="A1" pin="GND"/>
+<wire x1="-182.88" y1="0" x2="-182.88" y2="-5.08" width="0.1524" layer="91"/>
 </segment>
 <segment>
@@
 <net name="+12V" class="0">
 <segment>
-<pinref part="IC2" gate="G$1" pin="VIN"/>
 <wire x1="-195.58" y1="7.62" x2="-198.12" y2="7.62" width="0.1524" layer="91"/>
 <wire x1="-198.12" y1="7.62" x2="-205.74" y2="7.62" width="0.1524" layer="91"/>
@@
 <junction x="-205.74" y="7.62"/>
 <pinref part="SUPPLY9" gate="+12V" pin="+12V"/>
-</segment>
-</net>
+<pinref part="IC2" gate="A1" pin="VI"/>
+<wire x1="-195.58" y1="7.62" x2="-193.04" y2="7.62" width="0.1524" layer="91"/>
+</segment>
+</net>
