File: pov-globe2.sch (EAGLE design)
At the start: 82 parts, among them IC1 MEGA8-AI, IC2 7805DT, IC3 74595, IC4 74595, IC5 74595, IC6 74595, IC7 74595

Commit message: slot routing2
Changed lines of the file:
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@@
 <?xml version="1.0" encoding="utf-8"?>
 <!DOCTYPE eagle SYSTEM "eagle.dtd">
-<eagle version="6.4">
+<eagle version="6.6.0">
 <drawing>
 <settings>
@@
 <junction x="-167.64" y="-2.54"/>
 <junction x="-160.02" y="-2.54"/>
-</segment>
-<segment>
+<junction x="-182.88" y="0"/>
+</segment>
+<segment>
